File: tradfri_oled/tradfri_oled.kicad_pcb (KiCad board)
At the start: 2 copper layers, 14 parts, among them J1 tradfri_debugger, U1 TRADFRI, U2 LIS3DH

Commit message: 20200914
Parts:
- removed J1: tradfri_debugger, mybays_connector:debugger_2x05_P1.27mm_Vertical
- added CON1: CORTEX-DEBUGGER, mybays_connector:debugger_2x05_P1.27mm_Vertical, F.Cu at (146.5, 112.8)
- added D1: LED_RABG, mybays:SMD020RGBC, F.Cu at (106.5, 132.3)
- added J2: Conn_01x06, Connector_PinHeader_2.54mm:PinHeader_1x06_P2.54mm_Vertical, F.Cu at (104.9, 121.5)
- added J3: Conn_01x10, Connector_PinHeader_2.54mm:PinHeader_1x10_P2.54mm_Vertical, F.Cu at (140.6, 104.0)
- added J4: microusb, mybays_connector:MICRO-USB_MICRO-USB-17, F.Cu at (123.4, 146.3)
- added R6: R_US, Resistor_SMD:R_0603_1608Metric_Pad1.05x0.95mm_HandSolder, F.Cu at (104.0, 138.2)
- added R7: R_US, Resistor_SMD:R_0603_1608Metric_Pad1.05x0.95mm_HandSolder, F.Cu at (104.2, 141.1)
- added R8: R_US, Resistor_SMD:R_0603_1608Metric_Pad1.05x0.95mm_HandSolder, F.Cu at (104.3, 144.8)
- added U3: LM1117-3.3, myelin:SOT-223-LDO-1117LV, F.Cu at (138.7, 141.9)
- moved U2 33.2 mm to (145.9, 134.4), turned to 180 degrees
- moved OLED1 28.8 mm to (125.0, 124.0)
- moved U1 19.4 mm to (117.0, 112.1), turned to 90 degrees
Connections:
- U1 pad 1: Net-(U1-Pad1) -> GND
- U1 pad 10: Net-(U1-Pad10) -> /RESETn
- U1 pad 11: Net-(U1-Pad11) -> +3V3
- U1 pad 12: Net-(U1-Pad12) -> GND
- U1 pad 15: Net-(U1-Pad15) -> /I2C_SCL
- U1 pad 16: Net-(U1-Pad16) -> /I2C_SDA
- U1 pad 18: Net-(U1-Pad18) -> GND
- U1 pad 2: Net-(U1-Pad2) -> /UART_TX
- U1 pad 3: Net-(U1-Pad3) -> /UART_RX
- U1 pad 6: Net-(U1-Pad6) -> /DBG_SWCLK
- U1 pad 7: Net-(U1-Pad7) -> /DBG_SWDIO
- U1 pad 8: Net-(U1-Pad8) -> /DBG_SWO
- U1 pad 9: Net-(U1-Pad9) -> /DBG_TDI
Other:
- board outline added: 50 x 50 mm

Commit message: final
Parts:
- added C10: 470nf, Capacitor_SMD:C_0603_1608Metric_Pad1.05x0.95mm_HandSolder, F.Cu at (134.9, 136.1)
- added C11: 470nf, Capacitor_SMD:C_0603_1608Metric_Pad1.05x0.95mm_HandSolder, F.Cu at (115.0, 139.0)
- added C6: 4.7u, Capacitor_SMD:C_0603_1608Metric_Pad1.05x0.95mm_HandSolder, F.Cu at (147.0, 128.7)
- added C7: 4.7u, Capacitor_SMD:C_1206_3216Metric_Pad1.42x1.75mm_HandSolder, F.Cu at (132.9, 144.0)
- added C8: 4.7u, Capacitor_SMD:C_1206_3216Metric_Pad1.42x1.75mm_HandSolder, F.Cu at (146.7, 145.0)
- added C9: 470nf, Capacitor_SMD:C_0603_1608Metric_Pad1.05x0.95mm_HandSolder, F.Cu at (146.2, 103.8)
- added R10: 4.7k, Resistor_SMD:R_0402_1005Metric, F.Cu at (131.7, 136.1)
- added R9: 4.7k, Resistor_SMD:R_0402_1005Metric, F.Cu at (118.0, 139.0)
- added SW1: SW_Push, mybays_connector:turtlekey, B.Cu at (115.0, 139.0)
- added SW2: SW_Push, mybays_connector:turtlekey, B.Cu at (146.1, 103.8)
- added SW3: SW_Push, mybays_connector:turtlekey, B.Cu at (135.0, 139.0)
- D1: moved to B.Cu
- R2, R3, R4, R5: footprint Resistor_SMD:R_0603_1608Metric_Pad1.05x0.95mm_HandSolder -> Resistor_SMD:R_0402_1005Metric
- R6, R7, R8: value R_US -> 1k; footprint Resistor_SMD:R_0603_1608Metric_Pad1.05x0.95mm_HandSolder -> Resistor_SMD:R_0402_1005Metric
- moved R8 47.9 mm to (145.7, 120.7), turned to 90 degrees
- moved R6 45.5 mm to (147.8, 125.9), turned to 180 degrees
- moved R7 45.1 mm to (144.4, 120.7), turned to 90 degrees
- moved D1 40.8 mm to (146.5, 124.1), turned to 180 degrees
- moved C4 20.7 mm to (132.3, 128.7), turned to 90 degrees
- moved R5 19.3 mm to (146.5, 130.0), turned to 180 degrees
- moved R2 19.0 mm to (126.2, 127.0), turned to 270 degrees
- moved C3 16.2 mm to (134.2, 128.7), turned to 90 degrees
- moved C1 15.4 mm to (128.9, 128.4), turned to 90 degrees
- moved R3 13.8 mm to (123.6, 126.6), turned to 180 degrees
- moved R4 10.2 mm to (125.2, 127.0), turned to 270 degrees
- moved C5 9.04 mm to (114.2, 129.5), turned to 90 degrees
- moved C2 7.66 mm to (115.9, 129.5), turned to 90 degrees
- moved R1 7.66 mm to (117.7, 129.5), turned to 270 degrees
- moved U3 3.04 mm to (141.5, 143.0)
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Connections:
- net Net-(J2-Pad3) renamed /PB13
- net Net-(J2-Pad4) renamed /PB12
- CON1 pad 1: +5V -> Net-(CON1-Pad1)
- J3 pad 6: Net-(J3-Pad6) -> /PC11
- J3 pad 7: Net-(J3-Pad7) -> /PC10
- R6 pad 2: Net-(R6-Pad2) -> GND
- R7 pad 2: Net-(R7-Pad2) -> /DBG_TDI
- R8 pad 2: Net-(R8-Pad2) -> /DBG_SWO
- U1 pad 4: Net-(J3-Pad7) -> /PC10
- U1 pad 5: Net-(J3-Pad6) -> /PC11
- U2 pad 11: Net-(U2-Pad11) -> /PC11
- U2 pad 9: Net-(U2-Pad9) -> /PC10
Routing:
- net GND: track 0.00 -> 260.8 mm, vias 0 -> 14
- net +3V3: track 0.00 -> 154.1 mm, vias 0 -> 3
- net /I2C_SDA: track 0.00 -> 71.7 mm, vias 0 -> 1
- net /I2C_SCL: track 0.00 -> 66.3 mm, vias 0 -> 2
- net /PB12: track 0.00 -> 52.3 mm, vias 0 -> 1
- net /PB13: track 0.00 -> 38.3 mm, vias 0 -> 1
- net /DBG_SWO: track 0.00 -> 35.8 mm, vias 0 -> 1
- net /PC11: track 0.00 -> 33.7 mm, vias 0 -> 2
- net /RESETn: track 0.00 -> 32.0 mm
- net /DBG_TDI: track 0.00 -> 31.3 mm, vias 0 -> 2
- net /PC10: track 0.00 -> 30.2 mm, vias 0 -> 2
- net /UART_TX: track 0.00 -> 30.0 mm
- net /UART_RX: track 0.00 -> 27.3 mm
- net /DBG_SWDIO: track 0.00 -> 20.8 mm
- net /DBG_SWCLK: track 0.00 -> 20.0 mm
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- added copper zone on B.Cu, net GND
- added copper zone on F.Cu, net GND
Other:
- net class Default: clearance 0.2 -> 0.127; trace_width 0.25 -> 0.127
- rule trace_clearance: 0.2 -> 0.127
- rule trace_min: 0.2 -> 0.127
- board text added: "3V3"
- board text added: "B12"
- board text added: "B13"
- board text added: "GND"
- board text added: "PC10"
- board text added: "PC11"
- board text added: "RESET"
- board text added: "RX"
- board text added: "SCL"
- board text added: "SDA"
- board text added: "SWCLK"
- board text added: "SWDIO"
- board text added: "SWO"
- board text added: "TDI"
- board text added: "TX"
