File: tradfri_oled/tradfri_oled.sch (KiCad schematic (older format))
At the start: 14 parts, among them J1 tradfri_debugger, U1 TRADFRI, U2 LIS3DH

Commit message: 20200914
Parts:
- removed J1: tradfri_debugger, mybays_connector:debugger_2x05_P1.27mm_Vertical, symbol mybays_connector:tradfri_debugger
- added CON1: CORTEX-DEBUGGER, mybays_connector:debugger_2x05_P1.27mm_Vertical, symbol mybays_connector:CORTEX-DEBUGGER
- added D1: LED_RABG, mybays:SMD020RGBC, symbol Device:LED_RABG
- added J2: Conn_01x06, Connector_PinHeader_2.54mm:PinHeader_1x06_P2.54mm_Vertical, symbol Connector_Generic:Conn_01x06
- added J3: Conn_01x10, Connector_PinHeader_2.54mm:PinHeader_1x10_P2.54mm_Vertical, symbol Connector_Generic:Conn_01x10
- added J4: microusb, mybays_connector:MICRO-USB_MICRO-USB-17, symbol mybays_connector:microusb
- added R6, R7, R8: R_US, Resistor_SMD:R_0603_1608Metric_Pad1.05x0.95mm_HandSolder, symbol Device:R_US
- added U3: LM1117-3.3, myelin:SOT-223-LDO-1117LV, symbol Regulator_Linear:LM1117-3.3
Connections:
- net labels added: +5V, DBG_SWCLK, DBG_SWDIO, DBG_SWO, DBG_TDI, RESETn, UART_RX, UART_TX
- wire segments 77 -> 131
Other:
- moved on the sheet: R5, U1, U2

Commit message: final
Parts:
- added C10, C11, C9: 470nf, Capacitor_SMD:C_0603_1608Metric_Pad1.05x0.95mm_HandSolder, symbol Device:C
- added C6: 4.7u, Capacitor_SMD:C_0603_1608Metric_Pad1.05x0.95mm_HandSolder, symbol Device:C
- added C7, C8: 4.7u, Capacitor_SMD:C_1206_3216Metric_Pad1.42x1.75mm_HandSolder, symbol Device:C
- added R10, R9: 4.7k, Resistor_SMD:R_0402_1005Metric, symbol Device:R_US
- added SW1, SW2, SW3: SW_Push, mybays_connector:turtlekey, symbol Switch:SW_Push
- R2, R3, R4, R5: footprint Resistor_SMD:R_0603_1608Metric_Pad1.05x0.95mm_HandSolder -> Resistor_SMD:R_0402_1005Metric
- R6, R7, R8: value R_US -> 1k; footprint Resistor_SMD:R_0603_1608Metric_Pad1.05x0.95mm_HandSolder -> Resistor_SMD:R_0402_1005Metric
Connections:
- net labels added: PB12, PB13, PC10, PC11
- wire segments 131 -> 175
- no-connect marks 0 -> 9
